Commit message: april20

File: cylinder/urdf/cylinder.xacro (robot description, xacro)
@@ -1,5 +1,5 @@
 <?xml version="1.0"?>
 <robot name="cylinder" xmlns:xacro="http://www.ros.org/wiki/xacro">
-  <xacro:property name="humanRadius" value="0.3"/>
+  <xacro:property name="humanRadius" value="0.1"/>
   <xacro:property name="humanHeight" value="1.7"/>
   <xacro:property name="humanMass" value="100"/>
@@ -38,5 +38,5 @@
         <cylinder radius="${humanRadius}" length="${humanHeight}"/>
       </geometry>
-      <material name="orange"/>
+      <material name="green"/>
     </visual>
     <inertial>
@@ -47,5 +47,5 @@
   </link>
   <gazebo reference="human">
-    <material>Gazebo/Orange</material>
+    <material>Gazebo/Green</material>
   </gazebo>
 </robot>

File: cylinder/urdf/macros.xacro (robot description, xacro)
@@ -1,2 +1,3 @@
+<?xml version="1.0"?>
 <robot xmlns:xacro="http://www.ros.org/wiki/xacro">
   <xacro:macro name="cylinder_inertia" params="m r h">

File: mybot_description/urdf/macros.xacro (robot description, xacro)
@@ -1,3 +1,6 @@
+<?xml version="1.0"?>
 <robot xmlns:xacro="http://www.ros.org/wiki/xacro">
+  <xacro:property name="cameraPos" value="0.2"/>
+  <xacro:property name="cameraPosX" value="0.2"/>
   <xacro:macro name="cylinder_inertia" params="m r h">
     <inertia  ixx="${m*(3*r*r+h*h)/12}" ixy = "0" ixz = "0"
@@ -53,5 +56,5 @@
       <axis xyz="0 1 0" rpy="0 0 0" />
       <limit effort="100" velocity="100"/>
-      <joint_properties damping="0.0" friction="0.0"/>
+      <joint_properties damping="0.0" friction="0.1"/>
     </joint>
     <transmission name="${lr}_trans">

File: mybot_description/urdf/mybot.xacro (robot description, xacro)
@@ -6,5 +6,6 @@
   <xacro:property name="chassisWidth" value="0.2"/>
   <xacro:property name="chassisMass" value="50"/>
-  <xacro:property name="cameraPos" value="0.1"/>
+  <xacro:property name="cameraPos" value="0.2"/>
+  <xacro:property name="cameraPosX" value="0.2"/>
   <xacro:property name="casterRadius" value="0.05"/>
   <xacro:property name="casterMass" value="5"/>
@@ -18,10 +19,11 @@
   <xacro:include filename="$(find mybot_description)/urdf/materials.xacro" />
   <xacro:include filename="$(find mybot_description)/urdf/macros.xacro" />
+  <xacro:include filename="$(find mybot_description)/urdf/camera.gazebo" />
   <gazebo reference="chassis">
     <material>Gazebo/Orange</material>
   </gazebo>
   <gazebo reference="caster_wheel">
-    <mu1>0.0</mu1>
-    <mu2>0.0</mu2>
+    <mu1>1.0</mu1>
+    <mu2>1.0</mu2>
     <material>Gazebo/Red</material>
   </gazebo>
@@ -51,5 +53,5 @@
     </inertial>
   </link>
-  <joint name="joint1" type="fixed">
+  <joint name="fixed" type="fixed">
     <parent link="chassis"/>
     <child link="caster_wheel"/>
@@ -82,7 +84,6 @@
   </joint>
   <link name="camera">
-    <!-- pose value="0 1 0 0 -0 0" relative_to="" -->
     <collision>
-      <origin xyz="0 0 ${cameraPos}" rpy="0 0 0"/>
+      <origin xyz="${cameraPosX} 0 ${cameraPos}" rpy="0 0 0"/>
       <geometry>
         <box size="${cameraSize} ${cameraSize} ${cameraSize}"/>
@@ -90,5 +91,5 @@
     </collision>
     <visual>
-      <origin xyz="0 0 ${cameraPos}" rpy="0 0 0"/>
+      <origin xyz="${cameraPosX} 0 ${cameraPos}" rpy="0 0 0"/>
       <geometry>
         <box size="${cameraSize} ${cameraSize} ${cameraSize}"/>
@@ -98,5 +99,5 @@
     <inertial>
       <mass value="${cameraMass}"/>
-      <origin xyz="0 0 ${cameraPos}" rpy="0 0 0"/>
+      <origin xyz="${cameraPosX} 0 ${cameraPos}" rpy="0 0 0"/>
       <xacro:box_inertia m="${cameraMass}" x="${cameraSize}" y="${cameraSize}" z="${cameraSize}" />
     </inertial>
