Commit message: report final

File: mybot_description/urdf/macros.xacro (robot description, xacro)
@@ -1,6 +1,4 @@
 <?xml version="1.0"?>
 <robot xmlns:xacro="http://www.ros.org/wiki/xacro">
-  <xacro:property name="cameraPos" value="0.2"/>
-  <xacro:property name="cameraPosX" value="0.2"/>
   <xacro:macro name="cylinder_inertia" params="m r h">
     <inertia  ixx="${m*(3*r*r+h*h)/12}" ixy = "0" ixz = "0"
@@ -56,5 +54,5 @@
       <axis xyz="0 1 0" rpy="0 0 0" />
       <limit effort="100" velocity="100"/>
-      <joint_properties damping="0.0" friction="0.1"/>
+      <joint_properties damping="0.1" friction="0.5"/>
     </joint>
     <transmission name="${lr}_trans">

File: mybot_description/urdf/mybot.xacro (robot description, xacro)
@@ -15,5 +15,5 @@
   <xacro:property name="wheelMass" value="5"/>
   <xacro:property name="cameraSize" value="0.05"/>
-  <xacro:property name="cameraMass" value="0.1"/>
+  <xacro:property name="cameraMass" value="0.01"/>
   <xacro:include filename="$(find mybot_description)/urdf/mybot.gazebo" />
   <xacro:include filename="$(find mybot_description)/urdf/materials.xacro" />
